File: IO.kicad_sch (KiCad schematic)
At the start: 56 parts, among them J1 Connector, USB-TYPE-C-16P, J2 Conn_01x02, Q3 AO3400A, Q4 AO3401A, Q5 AO3401A, SW1 SK12D07VG4, U1 TPS63001DRCR, U2 TP4054

Commit message: First draft of layout done. Needs cleaning and DRC
Parts:
- added R28, R29: 10kΩ, PCM_JLCPCB:R_0402, symbol PCM_JLCPCB-Resistors:0402,10kΩ
- added U4: W25Q128, PCM_JLCPCB:SOIC-8_L5.3-W5.3-P1.27-LS8.0-BL, symbol PCM_JLCPCB-Memory:16MByte, SPI
Connections:
- net +3.3V: now also R28.1, R29.1, U4.8 (VCC)
- net CS: now also U4.1 (CS#)
- net GNDD: now also C13.2, U4.4 (GND)
- net LED_VDD: no longer C13.2
- net SPI.MISO: now also U4.2 (DO)
- net SPI.MOSI: now also U4.5 (DI)
- net SPI.SCK: now also U4.6 (CLK)
- new net IO2: R28.2, U4.3 (IO2)
- new net IO3: R29.2, U4.7 (IO3)
Other:
- note added: "-> No significant gain from power gating"
- note added: "Current draw"
- note added: "External flash"
- note added: "Power down ~1 uA Standby ~10 uA Read ~10 mA"
- note added: "Used for extra control or Quad SPI mode -> Not needed"
- moved on the sheet: C21, C22, Card1, D6, D7, Q4, Q5, R20, R21, R22, R23, SW1
