File: display.kicad_sch (KiCad schematic)
At the start: 32 parts, among them Q1 AO3401A, Q2 BSS138

Commit message: First draft of layout done. Needs cleaning and DRC
Changed lines of the file:
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@@
 		)
 	)
-	(hierarchical_label "SPI{SCK MOSI}"
+	(hierarchical_label "SPI{SCK MOSI MISO}"
 		(shape bidirectional)
 		(at 55.88 152.4 180)
